Commit message: Hier Mo 2

File: Bewegungsanalyse/catkin_ws/src/urdf_6_dofra_v3/urdf/URDF_Assembly_6_DOFRA_v3.urdf (robot description, URDF)
Before this commit: robot urdf_6_dofra_v3, 10 links, 9 joints
Links:
- removed link link1
- added link link_1, mass 0.98184; collision mesh filename=package://urdf_6_dofra_v3/meshes/link_1.STL; visual mesh filename=package://urdf_6_dofra_v3/meshes/link_1.STL
Joints:
- joint joint_1: child link1 -> link_1
- joint joint_2: parent link1 -> link_1

Commit message: Simulation Funktioniert endlich

File: Bewegungsanalyse/catkin_ws/src/urdf_6_dofra_v3/urdf/URDF_Assembly_6_DOFRA_v3.urdf (robot description, URDF)
Before this commit: robot urdf_6_dofra_v3, 9 links, 8 joints
Links:
- added link world
Joints:
- added joint world_joint: type fixed, parent world, child base_link, origin xyz=0 0 0 rpy=0 0 0
- joint joint_1: limit lower=-3.1416 upper=3.1416 effort=0 velocity=0 -> lower=-3.1416 upper=3.1416 effort=5 velocity=3.14
- joint joint_2: limit lower=-1.7453 upper=2.5307 effort=0 velocity=0 -> lower=-1.7453 upper=2.5307 effort=5 velocity=3.14
- joint joint_3: limit lower=-3.1416 upper=3.1416 effort=0 velocity=0 -> lower=-3.1416 upper=3.1416 effort=5 velocity=3.14
- joint joint_4: limit lower=-3.1416 upper=3.1416 effort=0 velocity=0 -> lower=-3.1416 upper=3.1416 effort=5 velocity=3.14
- joint joint_5: limit lower=-3.1416 upper=3.1416 effort=0 velocity=0 -> lower=-3.1416 upper=3.1416 effort=5 velocity=3.14
- joint joint_6: limit lower=-3.1416 upper=3.1416 effort=0 velocity=0 -> lower=-3.1416 upper=3.1416 effort=5 velocity=3.14
- joint linear_axis: limit lower=0 upper=1.3 effort=0 velocity=0 -> lower=0 upper=1.3 effort=5 velocity=3.14
