Commit message: working on gazebo-urdf with ros tutorial. See readme

File: Bewegungsanalyse/ros2_ws/src/descriptions/gripper/urdf/gripper.urdf.xacro (robot description, xacro)
@@ -5,5 +5,5 @@
 <robot name="gripper" xmlns:xacro="http://www.ros.org/wiki/xacro">
   <!-- Gazebo transmission interface -->
-  <xacro:include filename="$(find gripper)/urdf/gripper.transmission.xacro" />
+  <xacro:include filename="$(find gripper)/urdf/gripper_transmission.xacro" />
   <xacro:macro name="gripper" params="prefix"> <!-- parent-->
   <!-- is good like this, but for test cases outcommented -->
@@ -550,4 +550,7 @@
   </joint>
   </xacro:macro>
+  <!-- Call the gripper macro, just for now, when connectiong to robot call in top level .xacro -->
   <xacro:gripper prefix="gripper" /> <!-- parent-->
+  <!-- Call the transmission macro -->
+  <xacro:gripper_transmission prefix="gripper" />
 </robot>

File: Bewegungsanalyse/ros2_ws/src/descriptions/gripper/urdf/gripper_transmission.xacro (robot description, xacro)
@@ -2,4 +2,16 @@
 <robot xmlns:xacro="http://www.ros.org/wiki/xacro">
   <xacro:macro name="gripper_transmission" params="prefix">
+    <ros2_control name="GazeboSystem" type="system">
+    <hardware>
+      <plugin>gazebo_ros2_control/GazeboSystem</plugin>
+    </hardware>
+    <!-- List your joints here -->
+    <joint name="your_joint_name" />
+  </ros2_control>
+  <gazebo>
+    <plugin filename="libgazebo_ros2_control.so" name="gazebo_ros2_control">
+      <parameters>$(find gripper)/config/gazebo_ros2_control.yaml</parameters>
+    </plugin>
+  </gazebo>
     <!-- Transmission for gripper -->
     <transmission name="${prefix}_transmission">

Commit message: working on ros2 control

File: Bewegungsanalyse/ros2_ws/src/descriptions/gripper/urdf/gripper.urdf.xacro (robot description, xacro)
@@ -6,11 +6,11 @@
   <!-- Gazebo transmission interface -->
   <xacro:include filename="$(find gripper)/urdf/gripper_transmission.xacro" />
-  <xacro:macro name="gripper" params="prefix"> <!-- parent-->
+  <xacro:macro name="gripper" params="prefix parent"> <!-- parent-->
+  <link name="world" />
   <!-- is good like this, but for test cases outcommented -->
-    <!-- <joint name="${prefix}_base_joint" type="fixed">
+    <joint name="${prefix}_base_joint" type="fixed">
       <parent link="${parent}"/>
       <child link="${prefix}_mount_link"/>
-      <xacro:insert_block name="origin"/>
-    </joint> -->
+    </joint>
     <link
     name="${prefix}_mount_link">
@@ -108,9 +108,9 @@
       lower="-3.14"
       upper="3.14"
-      effort="1"
-      velocity="1" />
+      effort="1.0"
+      velocity="1.0" />
     <dynamics
-      damping="1"
-      friction="1" />
+      damping="1.0"
+      friction="1.0" />
     <mimic
       joint="${prefix}_joint_1_right"
@@ -173,9 +173,9 @@
       lower="-3.14"
       upper="3.14"
-      effort="1"
-      velocity="1" />
+      effort="1.0"
+      velocity="1.0" />
     <dynamics
-      damping="1"
-      friction="1" />
+      damping="1.0"
+      friction="1.0" />
     <mimic
       joint="${prefix}_joint_1_left"
@@ -237,6 +237,6 @@
     <limit
       lower="-3.14"
-      effort="0"
-      velocity="0" />
+      effort="0.0"
+      velocity="0.0" />
   </joint>
   <link
@@ -295,9 +295,9 @@
       lower="-3.14"
       upper="3.14"
-      effort="1"
-      velocity="1" />
+      effort="1.0"
+      velocity="1.0" />
     <dynamics
-      damping="1"
-      friction="1" />
+      damping="1.0"
+      friction="1.0" />
     <mimic
       joint="${prefix}_joint_1_left"
@@ -360,9 +360,9 @@
       lower="0"
       upper="1"
-      effort="1"
-      velocity="1" />
+      effort="1.0"
+      velocity="1.0" />
     <dynamics
-      damping="1"
-      friction="1" />
+      damping="1.0"
+      friction="1.0" />
   </joint>
   <link
@@ -421,9 +421,9 @@
       lower="-3.14"
       upper="3.14"
-      effort="1"
-      velocity="1" />
+      effort="1.0"
+      velocity="1.0" />
     <dynamics
-      damping="1"
-      friction="1" />
+      damping="1.0"
+      friction="1.0" />
     <mimic
       joint="${prefix}_joint_1_right"
@@ -539,9 +539,9 @@
       lower="-3.14"
       upper="3.14"
-      effort="1"
-      velocity="1" />
+      effort="1.0"
+      velocity="1.0" />
     <dynamics
-      damping="1"
-      friction="1" />
+      damping="1.0"
+      friction="1.0" />
     <mimic
       joint="${prefix}_joint_1_right"
@@ -551,5 +551,5 @@
   </xacro:macro>
   <!-- Call the gripper macro, just for now, when connectiong to robot call in top level .xacro -->
-  <xacro:gripper prefix="gripper" /> <!-- parent-->
+  <xacro:gripper prefix="gripper" parent="world" /> <!-- parent-->
   <!-- Call the transmission macro -->
   <xacro:gripper_transmission prefix="gripper" />
