Commit message: working on gazebo urdf spawn

File: Bewegungsanalyse/ros2_ws/src/descriptions/gripper/urdf/gripper_transmission.xacro (robot description, xacro)
@@ -2,17 +2,24 @@
 <robot xmlns:xacro="http://www.ros.org/wiki/xacro">
   <xacro:macro name="gripper_transmission" params="prefix">
-    <ros2_control name="GazeboSystem" type="system">
-    <hardware>
-      <plugin>gazebo_ros2_control/GazeboSystem</plugin>
-    </hardware>
-    <!-- List your joints here -->
-    <joint name="your_joint_name" />
-  </ros2_control>
-  <gazebo>
-    <plugin filename="libgazebo_ros2_control.so" name="gazebo_ros2_control">
-      <parameters>$(find gripper)/config/gazebo_ros2_control.yaml</parameters>
-    </plugin>
-  </gazebo>
-    <!-- Transmission for gripper -->
+    <!-- ROS 2 Control system -->
+    <ros2_control name="GripperSystem" type="system">
+      <hardware>
+        <plugin>gazebo_ros2_control/GazeboSystem</plugin>
+      </hardware>
+      <!-- Define joints controlled by ROS 2 control -->
+      <joint name="${prefix}_joint_1_right">
+        <command_interface name="position"/>
+        <state_interface name="position"/>
+        <state_interface name="velocity"/>
+      </joint>
+    </ros2_control>
+    <!-- Gazebo plugin for ROS 2 control -->
+    <gazebo>
+      <plugin filename="libgazebo_ros2_control.so" name="gazebo_ros2_control">
+        <robotSimType>gazebo_ros2_control/GazeboSystem</robotSimType>
+        <parameters>package://gripper/config/gazebo_ros2_control.yaml</parameters>
+      </plugin>
+    </gazebo>
+    <!-- Transmission for Gazebo -->
     <transmission name="${prefix}_transmission">
       <type>transmission_interface/SimpleTransmission</type>

Commit message: pushing current

File: Bewegungsanalyse/ros2_ws/src/descriptions/gripper/urdf/gripper_transmission.xacro (robot description, xacro)
@@ -5,5 +5,5 @@
     <ros2_control name="GripperSystem" type="system">
       <hardware>
-        <plugin>gazebo_ros2_control/GazeboSimSystem</plugin>
+        <plugin>gazebo_ros2_control/GazeboSystem</plugin>
       </hardware>
       <!-- Define joints controlled by ROS 2 control -->
@@ -16,23 +16,9 @@
     <!-- Gazebo plugin for ROS 2 control -->
     <gazebo>
-      <!-- <plugin filename="libgazebo_ros2_control.so" name="gazebo_ros2_control">
-        <robotSimType>gazebo_ros2_control/GazeboSystem</robotSimType>
-        <parameters>$(find gripper)/config/gazebo_ros2_control.yaml</parameters>
-      </plugin> -->
-      <plugin filename="libgazebo_ros2_control.so" name="gazebo_ros2_control">
-          <parameters>/app/install/gripper/share/gripper/config/gazebo_ros2_control.yaml</parameters>
-      </plugin>
+        <plugin name="gazebo_ros2_control" filename="libgazebo_ros2_control.so">
+            <robot_sim_type>gazebo_ros2_control/GazeboSystem</robot_sim_type>
+            <parameters>$(find gripper_moveit_config)/config/ros2_controllers.yaml</parameters>
+        </plugin>
     </gazebo>
-    <!-- Transmission for Gazebo
-    <transmission name="${prefix}_transmission">
-      <type>transmission_interface/SimpleTransmission</type>
-      <joint name="${prefix}_joint_1_right">
-        <hardwareInterface>hardware_interface/PositionJointInterface</hardwareInterface>
-      </joint>
-      <actuator name="${prefix}_actuator">
-        <hardwareInterface>hardware_interface/PositionJointInterface</hardwareInterface>
-        <mechanicalReduction>1.0</mechanicalReduction>
-      </actuator>
-    </transmission> -->
     <!-- Mimic joints for Gazebo -->
     <gazebo>
