Commit message: Save before replacing new base_link mesh

File: Bewegungsanalyse/ros2_ws/src/configs/six_dofra_config/config/urdf_6_dofra_v3.ros2_control.xacro (robot description, xacro)
@@ -2,5 +2,5 @@
 <robot xmlns:xacro="http://www.ros.org/wiki/xacro">
     <xacro:macro name="urdf_6_dofra_v3_ros2_control" params="name initial_positions_file">
-        <xacro:property name="initial_positions" value="${load_yaml(initial_positions_file)['initial_positions']}"/>
+        <xacro:property name="initial_positions" value="${xacro.load_yaml(initial_positions_file)['initial_positions']}"/>
         <ros2_control name="${name}" type="system">
             <hardware>

File: Bewegungsanalyse/ros2_ws/src/descriptions/urdf_6_dofra_v3/urdf/URDF_Assembly_6_DOFRA_v3.xacro (robot description, xacro)
@@ -19,14 +19,14 @@
             <origin xyz="0 0 0" rpy="0 0 0" />
             <geometry>
-                <mesh filename="package://urdf_6_dofra_v3/meshes/base_link.STL" />
-            </geometry>
-            <material name="">
-                <color rgba="0.79216 0.81961 0.93333 1" />
-            </material>
-        </visual>
-        <collision>
-            <origin xyz="0 0 0" rpy="0 0 0" />
-            <geometry>
-                <mesh filename="package://urdf_6_dofra_v3/meshes/base_link.STL" />
+                <mesh filename="file://$(find urdf_6_dofra_v3)/meshes/base_link.STL" />
+            </geometry>
+            <material name="">
+                <color rgba="0.79216 0.81961 0.93333 1" />
+            </material>
+        </visual>
+        <collision>
+            <origin xyz="0 0 0" rpy="0 0 0" />
+            <geometry>
+                <mesh filename="file://$(find urdf_6_dofra_v3)/meshes/base_link.STL" />
             </geometry>
         </collision>
@@ -41,14 +41,14 @@
             <origin xyz="0 0 0" rpy="0 0 0" />
             <geometry>
-                <mesh filename="package://urdf_6_dofra_v3/meshes/linear_sledge.STL" />
-            </geometry>
-            <material name="">
-                <color rgba="0.79216 0.81961 0.93333 1" />
-            </material>
-        </visual>
-        <collision>
-            <origin xyz="0 0 0" rpy="0 0 0" />
-            <geometry>
-                <mesh filename="package://urdf_6_dofra_v3/meshes/linear_sledge.STL" />
+                <mesh filename="file://$(find urdf_6_dofra_v3)/meshes/linear_sledge.STL" />
+            </geometry>
+            <material name="">
+                <color rgba="0.79216 0.81961 0.93333 1" />
+            </material>
+        </visual>
+        <collision>
+            <origin xyz="0 0 0" rpy="0 0 0" />
+            <geometry>
+                <mesh filename="file://$(find urdf_6_dofra_v3)/meshes/linear_sledge.STL" />
             </geometry>
         </collision>
@@ -71,14 +71,14 @@
             <origin xyz="0 0 0" rpy="0 0 0" />
             <geometry>
-                <mesh filename="package://urdf_6_dofra_v3/meshes/link_0.STL" />
-            </geometry>
-            <material name="">
-                <color rgba="0.79216 0.81961 0.93333 1" />
-            </material>
-        </visual>
-        <collision>
-            <origin xyz="0 0 0" rpy="0 0 0" />
-            <geometry>
-                <mesh filename="package://urdf_6_dofra_v3/meshes/link_0.STL" />
+                <mesh filename="file://$(find urdf_6_dofra_v3)/meshes/link_0.STL" />
+            </geometry>
+            <material name="">
+                <color rgba="0.79216 0.81961 0.93333 1" />
+            </material>
+        </visual>
+        <collision>
+            <origin xyz="0 0 0" rpy="0 0 0" />
+            <geometry>
+                <mesh filename="file://$(find urdf_6_dofra_v3)/meshes/link_0.STL" />
             </geometry>
         </collision>
@@ -99,14 +99,14 @@
             <origin xyz="0 0 0" rpy="0 0 0" />
             <geometry>
-                <mesh filename="package://urdf_6_dofra_v3/meshes/link_1.STL" />
-            </geometry>
-            <material name="">
-                <color rgba="0.79216 0.81961 0.93333 1" />
-            </material>
-        </visual>
-        <collision>
-            <origin xyz="0 0 0" rpy="0 0 0" />
-            <geometry>
-                <mesh filename="package://urdf_6_dofra_v3/meshes/link_1.STL" />
+                <mesh filename="file://$(find urdf_6_dofra_v3)/meshes/link_1.STL" />
+            </geometry>
+            <material name="">
+                <color rgba="0.79216 0.81961 0.93333 1" />
+            </material>
+        </visual>
+        <collision>
+            <origin xyz="0 0 0" rpy="0 0 0" />
+            <geometry>
+                <mesh filename="file://$(find urdf_6_dofra_v3)/meshes/link_1.STL" />
             </geometry>
         </collision>
@@ -129,14 +129,14 @@
             <origin xyz="0 0 0" rpy="0 0 0" />
             <geometry>
-                <mesh filename="package://urdf_6_dofra_v3/meshes/link_2.STL" />
-            </geometry>
-            <material name="">
-                <color rgba="0.79216 0.81961 0.93333 1" />
-            </material>
-        </visual>
-        <collision>
-            <origin xyz="0 0 0" rpy="0 0 0" />
-            <geometry>
-                <mesh filename="package://urdf_6_dofra_v3/meshes/link_2.STL" />
+                <mesh filename="file://$(find urdf_6_dofra_v3)/meshes/link_2.STL" />
+            </geometry>
+            <material name="">
+                <color rgba="0.79216 0.81961 0.93333 1" />
+            </material>
+        </visual>
+        <collision>
+            <origin xyz="0 0 0" rpy="0 0 0" />
+            <geometry>
+                <mesh filename="file://$(find urdf_6_dofra_v3)/meshes/link_2.STL" />
             </geometry>
         </collision>
@@ -159,5 +159,5 @@
             <origin xyz="0 0 0" rpy="0 0 0" />
             <geometry>
-                <mesh filename="package://urdf_6_dofra_v3/meshes/link_3.STL" />
+                <mesh filename="file://$(find urdf_6_dofra_v3)/meshes/link_3.STL" />
             </geometry>
             <material name="">
@@ -168,5 +168,5 @@
             <origin xyz="0 0 0" rpy="0 0 0" />
             <geometry>
-                <mesh filename="package://urdf_6_dofra_v3/meshes/link_3.STL" />
+                <mesh filename="file://$(find urdf_6_dofra_v3)/meshes/link_3.STL" />
             </geometry>
         </collision>
@@ -189,5 +189,5 @@
             <origin xyz="0 0 0" rpy="0 0 0" />
             <geometry>
-                <mesh filename="package://urdf_6_dofra_v3/meshes/link_4.STL" />
+                <mesh filename="file://$(find urdf_6_dofra_v3)/meshes/link_4.STL" />
             </geometry>
             <material name="">
@@ -198,5 +198,5 @@
             <origin xyz="0 0 0" rpy="0 0 0" />
             <geometry>
-                <mesh filename="package://urdf_6_dofra_v3/meshes/link_4.STL" />
+                <mesh filename="file://$(find urdf_6_dofra_v3)/meshes/link_4.STL" />
             </geometry>
         </collision>
@@ -219,5 +219,5 @@
             <origin xyz="0 0 0" rpy="0 0 0" />
             <geometry>
-                <mesh filename="package://urdf_6_dofra_v3/meshes/link_5.STL" />
+                <mesh filename="file://$(find urdf_6_dofra_v3)/meshes/link_5.STL" />
             </geometry>
             <material name="">
@@ -228,5 +228,5 @@
             <origin xyz="0 0 0" rpy="0 0 0" />
             <geometry>
-                <mesh filename="package://urdf_6_dofra_v3/meshes/link_5.STL" />
+                <mesh filename="file://$(find urdf_6_dofra_v3)/meshes/link_5.STL" />
             </geometry>
         </collision>
@@ -249,5 +249,5 @@
             <origin xyz="0 0 0" rpy="0 0 0" />
             <geometry>
-                <mesh filename="package://urdf_6_dofra_v3/meshes/link_6.STL" />
+                <mesh filename="file://$(find urdf_6_dofra_v3)/meshes/link_6.STL" />
             </geometry>
             <material name="">
@@ -258,5 +258,5 @@
             <origin xyz="0 0 0" rpy="0 0 0" />
             <geometry>
-                <mesh filename="package://urdf_6_dofra_v3/meshes/link_6.STL" />
+                <mesh filename="file://$(find urdf_6_dofra_v3)/meshes/link_6.STL" />
             </geometry>
         </collision>

File: Bewegungsanalyse/ros2_ws/src/simulations/six_dofra_gazebo/urdf/six_dofra_gazebo.xacro (robot description, xacro)
@@ -3,5 +3,5 @@
      Commit Version: 1.6.0-4-g7f85cfe  Build Version: 1.6.7995.38578
      For more information, please see http://wiki.ros.org/sw_urdf_exporter -->
-<robot xmlns:xacro="http://www.ros.org/wiki/xacro" name="urdf_6_dofra_v3">
+<robot xmlns:xacro="http://www.ros.org/wiki/xacro" name="six_dofra_gazebo">
     <link name="world"/>
     <joint name="world_joint" type="fixed">
@@ -19,14 +19,14 @@
             <origin xyz="0 0 0" rpy="0 0 0" />
             <geometry>
-                <mesh filename="package://urdf_6_dofra_v3/meshes/base_link.STL" />
-            </geometry>
-            <material name="">
-                <color rgba="0.79216 0.81961 0.93333 1" />
-            </material>
-        </visual>
-        <collision>
-            <origin xyz="0 0 0" rpy="0 0 0" />
-            <geometry>
-                <mesh filename="package://urdf_6_dofra_v3/meshes/base_link.STL" />
+                <mesh filename="package://six_dofra_gazebo/meshes/base_link.STL" />
+            </geometry>
+            <material name="">
+                <color rgba="0.79216 0.81961 0.93333 1" />
+            </material>
+        </visual>
+        <collision>
+            <origin xyz="0 0 0" rpy="0 0 0" />
+            <geometry>
+                <mesh filename="package://six_dofra_gazebo/meshes/base_link.STL" />
             </geometry>
         </collision>
@@ -41,14 +41,14 @@
             <origin xyz="0 0 0" rpy="0 0 0" />
             <geometry>
-                <mesh filename="package://urdf_6_dofra_v3/meshes/linear_sledge.STL" />
-            </geometry>
-            <material name="">
-                <color rgba="0.79216 0.81961 0.93333 1" />
-            </material>
-        </visual>
-        <collision>
-            <origin xyz="0 0 0" rpy="0 0 0" />
-            <geometry>
-                <mesh filename="package://urdf_6_dofra_v3/meshes/linear_sledge.STL" />
+                <mesh filename="package://six_dofra_gazebo/meshes/linear_sledge.STL" />
+            </geometry>
+            <material name="">
+                <color rgba="0.79216 0.81961 0.93333 1" />
+            </material>
+        </visual>
+        <collision>
+            <origin xyz="0 0 0" rpy="0 0 0" />
+            <geometry>
+                <mesh filename="package://six_dofra_gazebo/meshes/linear_sledge.STL" />
             </geometry>
         </collision>
@@ -71,14 +71,14 @@
             <origin xyz="0 0 0" rpy="0 0 0" />
             <geometry>
-                <mesh filename="package://urdf_6_dofra_v3/meshes/link_0.STL" />
-            </geometry>
-            <material name="">
-                <color rgba="0.79216 0.81961 0.93333 1" />
-            </material>
-        </visual>
-        <collision>
-            <origin xyz="0 0 0" rpy="0 0 0" />
-            <geometry>
-                <mesh filename="package://urdf_6_dofra_v3/meshes/link_0.STL" />
+                <mesh filename="package://six_dofra_gazebo/meshes/link_0.STL" />
+            </geometry>
+            <material name="">
+                <color rgba="0.79216 0.81961 0.93333 1" />
+            </material>
+        </visual>
+        <collision>
+            <origin xyz="0 0 0" rpy="0 0 0" />
+            <geometry>
+                <mesh filename="package://six_dofra_gazebo/meshes/link_0.STL" />
             </geometry>
         </collision>
@@ -99,14 +99,14 @@
             <origin xyz="0 0 0" rpy="0 0 0" />
             <geometry>
-                <mesh filename="package://urdf_6_dofra_v3/meshes/link_1.STL" />
-            </geometry>
-            <material name="">
-                <color rgba="0.79216 0.81961 0.93333 1" />
-            </material>
-        </visual>
-        <collision>
-            <origin xyz="0 0 0" rpy="0 0 0" />
-            <geometry>
-                <mesh filename="package://urdf_6_dofra_v3/meshes/link_1.STL" />
+                <mesh filename="package://six_dofra_gazebo/meshes/link_1.STL" />
+            </geometry>
+            <material name="">
+                <color rgba="0.79216 0.81961 0.93333 1" />
+            </material>
+        </visual>
+        <collision>
+            <origin xyz="0 0 0" rpy="0 0 0" />
+            <geometry>
+                <mesh filename="package://six_dofra_gazebo/meshes/link_1.STL" />
             </geometry>
         </collision>
@@ -129,14 +129,14 @@
             <origin xyz="0 0 0" rpy="0 0 0" />
             <geometry>
-                <mesh filename="package://urdf_6_dofra_v3/meshes/link_2.STL" />
-            </geometry>
-            <material name="">
-                <color rgba="0.79216 0.81961 0.93333 1" />
-            </material>
-        </visual>
-        <collision>
-            <origin xyz="0 0 0" rpy="0 0 0" />
-            <geometry>
-                <mesh filename="package://urdf_6_dofra_v3/meshes/link_2.STL" />
+                <mesh filename="package://six_dofra_gazebo/meshes/link_2.STL" />
+            </geometry>
+            <material name="">
+                <color rgba="0.79216 0.81961 0.93333 1" />
+            </material>
+        </visual>
+        <collision>
+            <origin xyz="0 0 0" rpy="0 0 0" />
+            <geometry>
+                <mesh filename="package://six_dofra_gazebo/meshes/link_2.STL" />
             </geometry>
         </collision>
@@ -159,5 +159,5 @@
             <origin xyz="0 0 0" rpy="0 0 0" />
             <geometry>
-                <mesh filename="package://urdf_6_dofra_v3/meshes/link_3.STL" />
+                <mesh filename="package://six_dofra_gazebo/meshes/link_3.STL" />
             </geometry>
             <material name="">
@@ -168,5 +168,5 @@
             <origin xyz="0 0 0" rpy="0 0 0" />
             <geometry>
-                <mesh filename="package://urdf_6_dofra_v3/meshes/link_3.STL" />
+                <mesh filename="package://six_dofra_gazebo/meshes/link_3.STL" />
             </geometry>
         </collision>
@@ -189,5 +189,5 @@
             <origin xyz="0 0 0" rpy="0 0 0" />
             <geometry>
-                <mesh filename="package://urdf_6_dofra_v3/meshes/link_4.STL" />
+                <mesh filename="package://six_dofra_gazebo/meshes/link_4.STL" />
             </geometry>
             <material name="">
@@ -198,5 +198,5 @@
             <origin xyz="0 0 0" rpy="0 0 0" />
             <geometry>
-                <mesh filename="package://urdf_6_dofra_v3/meshes/link_4.STL" />
+                <mesh filename="package://six_dofra_gazebo/meshes/link_4.STL" />
             </geometry>
         </collision>
@@ -219,5 +219,5 @@
             <origin xyz="0 0 0" rpy="0 0 0" />
             <geometry>
-                <mesh filename="package://urdf_6_dofra_v3/meshes/link_5.STL" />
+                <mesh filename="package://six_dofra_gazebo/meshes/link_5.STL" />
             </geometry>
             <material name="">
@@ -228,5 +228,5 @@
             <origin xyz="0 0 0" rpy="0 0 0" />
             <geometry>
-                <mesh filename="package://urdf_6_dofra_v3/meshes/link_5.STL" />
+                <mesh filename="package://six_dofra_gazebo/meshes/link_5.STL" />
             </geometry>
         </collision>
@@ -249,5 +249,5 @@
             <origin xyz="0 0 0" rpy="0 0 0" />
             <geometry>
-                <mesh filename="package://urdf_6_dofra_v3/meshes/link_6.STL" />
+                <mesh filename="package://six_dofra_gazebo/meshes/link_6.STL" />
             </geometry>
             <material name="">
@@ -258,5 +258,5 @@
             <origin xyz="0 0 0" rpy="0 0 0" />
             <geometry>
-                <mesh filename="package://urdf_6_dofra_v3/meshes/link_6.STL" />
+                <mesh filename="package://six_dofra_gazebo/meshes/link_6.STL" />
             </geometry>
         </collision>
