Commit message: New description package for six_dofra

File: Bewegungsanalyse/ros2_ws/src/descriptions/six_dofra_description/urdf/six_dofra_description.urdf (robot description, URDF)
Before this commit: robot urdf_6_dofra_v3, 10 links, 9 joints
Links:
- link base_link: geometry collision mesh filename=package://six_dofra_description/meshes/base_link.STL; visual mesh filename=package://six_dofra_description/meshes/base_link.STL
- link linear_sledge: geometry collision mesh filename=package://six_dofra_description/meshes/linear_sledge.STL; visual mesh filename=package://six_dofra_description/meshes/linear_sledge.STL
- link link_0: geometry collision mesh filename=package://six_dofra_description/meshes/link_0.STL; visual mesh filename=package://six_dofra_description/meshes/link_0.STL
- link link_1: geometry collision mesh filename=package://six_dofra_description/meshes/link_1.STL; visual mesh filename=package://six_dofra_description/meshes/link_1.STL
- link link_2: geometry collision mesh filename=package://six_dofra_description/meshes/link_2.STL; visual mesh filename=package://six_dofra_description/meshes/link_2.STL
- link link_3: geometry collision mesh filename=package://six_dofra_description/meshes/link_3.STL; visual mesh filename=package://six_dofra_description/meshes/link_3.STL
- link link_4: geometry collision mesh filename=package://six_dofra_description/meshes/link_4.STL; visual mesh filename=package://six_dofra_description/meshes/link_4.STL
- link link_5: geometry collision mesh filename=package://six_dofra_description/meshes/link_5.STL; visual mesh filename=package://six_dofra_description/meshes/link_5.STL
- link link_6: geometry collision mesh filename=package://six_dofra_description/meshes/link_6.STL; visual mesh filename=package://six_dofra_description/meshes/link_6.STL

File: Bewegungsanalyse/ros2_ws/src/descriptions/six_dofra_description/urdf/six_dofra_description.urdf.xacro (robot description, xacro)
@@ -3,5 +3,5 @@
      Commit Version: 1.6.0-4-g7f85cfe  Build Version: 1.6.7995.38578
      For more information, please see http://wiki.ros.org/sw_urdf_exporter -->
-<robot xmlns:xacro="http://www.ros.org/wiki/xacro" name="urdf_6_dofra_v3">
+<robot xmlns:xacro="http://www.ros.org/wiki/xacro" name="six_dofra_description">
     <link name="world"/>
     <joint name="world_joint" type="fixed">
@@ -19,14 +19,14 @@
             <origin xyz="0 0 0" rpy="0 0 0" />
             <geometry>
-                <mesh filename="file://$(find urdf_6_dofra_v3)/meshes/base_link.STL" />
-            </geometry>
-            <material name="">
-                <color rgba="0.79216 0.81961 0.93333 1" />
-            </material>
-        </visual>
-        <collision>
-            <origin xyz="0 0 0" rpy="0 0 0" />
-            <geometry>
-                <mesh filename="file://$(find urdf_6_dofra_v3)/meshes/base_link.STL" />
+                <mesh filename="file://$(find six_dofra_description)/meshes/base_link.STL" />
+            </geometry>
+            <material name="">
+                <color rgba="0.79216 0.81961 0.93333 1" />
+            </material>
+        </visual>
+        <collision>
+            <origin xyz="0 0 0" rpy="0 0 0" />
+            <geometry>
+                <mesh filename="file://$(find six_dofra_description)/meshes/base_link.STL" />
             </geometry>
         </collision>
@@ -41,14 +41,14 @@
             <origin xyz="0 0 0" rpy="0 0 0" />
             <geometry>
-                <mesh filename="file://$(find urdf_6_dofra_v3)/meshes/linear_sledge.STL" />
-            </geometry>
-            <material name="">
-                <color rgba="0.79216 0.81961 0.93333 1" />
-            </material>
-        </visual>
-        <collision>
-            <origin xyz="0 0 0" rpy="0 0 0" />
-            <geometry>
-                <mesh filename="file://$(find urdf_6_dofra_v3)/meshes/linear_sledge.STL" />
+                <mesh filename="file://$(find six_dofra_description)/meshes/linear_sledge.STL" />
+            </geometry>
+            <material name="">
+                <color rgba="0.79216 0.81961 0.93333 1" />
+            </material>
+        </visual>
+        <collision>
+            <origin xyz="0 0 0" rpy="0 0 0" />
+            <geometry>
+                <mesh filename="file://$(find six_dofra_description)/meshes/linear_sledge.STL" />
             </geometry>
         </collision>
@@ -71,14 +71,14 @@
             <origin xyz="0 0 0" rpy="0 0 0" />
             <geometry>
-                <mesh filename="file://$(find urdf_6_dofra_v3)/meshes/link_0.STL" />
-            </geometry>
-            <material name="">
-                <color rgba="0.79216 0.81961 0.93333 1" />
-            </material>
-        </visual>
-        <collision>
-            <origin xyz="0 0 0" rpy="0 0 0" />
-            <geometry>
-                <mesh filename="file://$(find urdf_6_dofra_v3)/meshes/link_0.STL" />
+                <mesh filename="file://$(find six_dofra_description)/meshes/link_0.STL" />
+            </geometry>
+            <material name="">
+                <color rgba="0.79216 0.81961 0.93333 1" />
+            </material>
+        </visual>
+        <collision>
+            <origin xyz="0 0 0" rpy="0 0 0" />
+            <geometry>
+                <mesh filename="file://$(find six_dofra_description)/meshes/link_0.STL" />
             </geometry>
         </collision>
@@ -99,14 +99,14 @@
             <origin xyz="0 0 0" rpy="0 0 0" />
             <geometry>
-                <mesh filename="file://$(find urdf_6_dofra_v3)/meshes/link_1.STL" />
-            </geometry>
-            <material name="">
-                <color rgba="0.79216 0.81961 0.93333 1" />
-            </material>
-        </visual>
-        <collision>
-            <origin xyz="0 0 0" rpy="0 0 0" />
-            <geometry>
-                <mesh filename="file://$(find urdf_6_dofra_v3)/meshes/link_1.STL" />
+                <mesh filename="file://$(find six_dofra_description)/meshes/link_1.STL" />
+            </geometry>
+            <material name="">
+                <color rgba="0.79216 0.81961 0.93333 1" />
+            </material>
+        </visual>
+        <collision>
+            <origin xyz="0 0 0" rpy="0 0 0" />
+            <geometry>
+                <mesh filename="file://$(find six_dofra_description)/meshes/link_1.STL" />
             </geometry>
         </collision>
@@ -129,14 +129,14 @@
             <origin xyz="0 0 0" rpy="0 0 0" />
             <geometry>
-                <mesh filename="file://$(find urdf_6_dofra_v3)/meshes/link_2.STL" />
-            </geometry>
-            <material name="">
-                <color rgba="0.79216 0.81961 0.93333 1" />
-            </material>
-        </visual>
-        <collision>
-            <origin xyz="0 0 0" rpy="0 0 0" />
-            <geometry>
-                <mesh filename="file://$(find urdf_6_dofra_v3)/meshes/link_2.STL" />
+                <mesh filename="file://$(find six_dofra_description)/meshes/link_2.STL" />
+            </geometry>
+            <material name="">
+                <color rgba="0.79216 0.81961 0.93333 1" />
+            </material>
+        </visual>
+        <collision>
+            <origin xyz="0 0 0" rpy="0 0 0" />
+            <geometry>
+                <mesh filename="file://$(find six_dofra_description)/meshes/link_2.STL" />
             </geometry>
         </collision>
@@ -159,5 +159,5 @@
             <origin xyz="0 0 0" rpy="0 0 0" />
             <geometry>
-                <mesh filename="file://$(find urdf_6_dofra_v3)/meshes/link_3.STL" />
+                <mesh filename="file://$(find six_dofra_description)/meshes/link_3.STL" />
             </geometry>
             <material name="">
@@ -168,5 +168,5 @@
             <origin xyz="0 0 0" rpy="0 0 0" />
             <geometry>
-                <mesh filename="file://$(find urdf_6_dofra_v3)/meshes/link_3.STL" />
+                <mesh filename="file://$(find six_dofra_description)/meshes/link_3.STL" />
             </geometry>
         </collision>
@@ -189,5 +189,5 @@
             <origin xyz="0 0 0" rpy="0 0 0" />
             <geometry>
-                <mesh filename="file://$(find urdf_6_dofra_v3)/meshes/link_4.STL" />
+                <mesh filename="file://$(find six_dofra_description)/meshes/link_4.STL" />
             </geometry>
             <material name="">
@@ -198,5 +198,5 @@
             <origin xyz="0 0 0" rpy="0 0 0" />
             <geometry>
-                <mesh filename="file://$(find urdf_6_dofra_v3)/meshes/link_4.STL" />
+                <mesh filename="file://$(find six_dofra_description)/meshes/link_4.STL" />
             </geometry>
         </collision>
@@ -219,5 +219,5 @@
             <origin xyz="0 0 0" rpy="0 0 0" />
             <geometry>
-                <mesh filename="file://$(find urdf_6_dofra_v3)/meshes/link_5.STL" />
+                <mesh filename="file://$(find six_dofra_description)/meshes/link_5.STL" />
             </geometry>
             <material name="">
@@ -228,5 +228,5 @@
             <origin xyz="0 0 0" rpy="0 0 0" />
             <geometry>
-                <mesh filename="file://$(find urdf_6_dofra_v3)/meshes/link_5.STL" />
+                <mesh filename="file://$(find six_dofra_description)/meshes/link_5.STL" />
             </geometry>
         </collision>
@@ -249,5 +249,5 @@
             <origin xyz="0 0 0" rpy="0 0 0" />
             <geometry>
-                <mesh filename="file://$(find urdf_6_dofra_v3)/meshes/link_6.STL" />
+                <mesh filename="file://$(find six_dofra_description)/meshes/link_6.STL" />
             </geometry>
             <material name="">
@@ -258,5 +258,5 @@
             <origin xyz="0 0 0" rpy="0 0 0" />
             <geometry>
-                <mesh filename="file://$(find urdf_6_dofra_v3)/meshes/link_6.STL" />
+                <mesh filename="file://$(find six_dofra_description)/meshes/link_6.STL" />
             </geometry>
         </collision>
