Commit message: Robot+Gripper config created, but not working

File: Bewegungsanalyse/ros2_ws/src/descriptions/six_dofra_description/urdf/six_dofra_description.urdf.xacro (robot description, xacro)
@@ -270,4 +270,10 @@
         <dynamics damping="0.01" friction="0.01" />
     </joint>
+    <link name="tool_nullframe_link"></link>
+    <joint name="tool_nullframe_joint" type="fixed">
+        <origin xyz="0 0 0.01" rpy="0 0 0" />
+        <parent link="link_6"/>
+        <child link="tool_nullframe_link"/>
+    </joint>
     <transmission name="trans_linear_axis">
         <type>transmission_interface/SimpleTransmission</type>

Commit message: Shinra Tensei

File: Bewegungsanalyse/ros2_ws/src/descriptions/six_dofra_description/urdf/six_dofra_description.urdf.xacro (robot description, xacro)
@@ -1,6 +1,3 @@
-<?xml version="1.0" encoding="utf-8" ?>
-<!-- This URDF was automatically created by SolidWorks to URDF Exporter! Originally created by Stephen Brawner (brawner@gmail.com)
-     Commit Version: 1.6.0-4-g7f85cfe  Build Version: 1.6.7995.38578
-     For more information, please see http://wiki.ros.org/sw_urdf_exporter -->
+<?xml version="1.0"?>
 <robot xmlns:xacro="http://www.ros.org/wiki/xacro" name="six_dofra_description">
     <link name="world"/>
@@ -61,4 +58,5 @@
         <limit lower="0" upper="1.3" effort="5" velocity="3.14" />
         <dynamics damping="0.01" friction="0.01" />
+        <hardwareInterface>Position</hardwareInterface>
     </joint>
     <link name="link_0">
@@ -119,4 +117,5 @@
         <limit lower="-3.1416" upper="3.1416" effort="5" velocity="3.14" />
         <dynamics damping="0.01" friction="0.01" />
+        <hardwareInterface>Position</hardwareInterface>
     </joint>
     <link name="link_2">
@@ -149,4 +148,5 @@
         <limit lower="-1.7453" upper="2.5307" effort="5" velocity="3.14" />
         <dynamics damping="0.01" friction="0.01" />
+        <hardwareInterface>Position</hardwareInterface>
     </joint>
     <link name="link_3">
@@ -179,4 +179,5 @@
         <limit lower="-3.1416" upper="3.1416" effort="5" velocity="3.14" />
         <dynamics damping="0.01" friction="0.01" />
+        <hardwareInterface>Position</hardwareInterface>
     </joint>
     <link name="link_4">
@@ -209,4 +210,5 @@
         <limit lower="-3.1416" upper="3.1416" effort="5" velocity="3.14" />
         <dynamics damping="0.01" friction="0.01" />
+        <hardwareInterface>Position</hardwareInterface>
     </joint>
     <link name="link_5">
@@ -239,4 +241,5 @@
         <limit lower="-3.1416" upper="3.1416" effort="5" velocity="3.14" />
         <dynamics damping="0.01" friction="0.01" />
+        <hardwareInterface>Position</hardwareInterface>
     </joint>
     <link name="link_6">
@@ -269,4 +272,5 @@
         <limit lower="-3.1416" upper="3.1416" effort="5" velocity="3.14" />
         <dynamics damping="0.01" friction="0.01" />
+        <hardwareInterface>Position</hardwareInterface>
     </joint>
     <link name="tool_nullframe_link"></link>
@@ -276,122 +280,93 @@
         <child link="tool_nullframe_link"/>
     </joint>
-    <transmission name="trans_linear_axis">
-        <type>transmission_interface/SimpleTransmission</type>
+    <!-- <ros2_control name="GazeboSystem" type="system"> -->
+    <ros2_control name="six_dofra_description" type="system">
+        <hardware>
+            <plugin>gazebo_ros2_control/GazeboSystem</plugin>
+        </hardware>
+        <!-- ros2 control commands for linear_axis -->
         <joint name="linear_axis">
-            <hardwareInterface>hardware_interface/PositionJointInterface</hardwareInterface>
-        </joint>
-        <actuator name="linear_axis_motor">
-            <hardwareInterface>hardware_interface/PositionJointInterface</hardwareInterface>
-            <mechanicalReduction>1</mechanicalReduction>
-        </actuator>
-    </transmission>
-    <transmission name="trans_joint_1">
-        <type>transmission_interface/SimpleTransmission</type>
+            <command_interface name="position">
+                <param name="min">-3.14</param>
+                <param name="max">3.14</param>
+            </command_interface>
+            <state_interface name="position">
+                <param name="initial_value">0.0</param>
+            </state_interface>
+            <state_interface name="velocity"/>
+            <state_interface name="effort"/>
+        </joint>
+        <!-- ros2 control commands for joint_1 -->
         <joint name="joint_1">
-            <hardwareInterface>hardware_interface/PositionJointInterface</hardwareInterface>
-        </joint>
-        <actuator name="joint_1_motor">
-            <hardwareInterface>hardware_interface/PositionJointInterface</hardwareInterface>
-            <mechanicalReduction>1</mechanicalReduction>
-        </actuator>
-    </transmission>
-    <transmission name="trans_joint_2">
-        <type>transmission_interface/SimpleTransmission</type>
+        <command_interface name="position">
+            <param name="min">-3.14</param>
+            <param name="max">3.14</param>
+        </command_interface>
+        <state_interface name="position">
+                <param name="initial_value">0.0</param>
+                </state_interface>
+        <state_interface name="velocity"/>
+        <state_interface name="effort"/>
+        </joint>
         <joint name="joint_2">
-            <hardwareInterface>hardware_interface/PositionJointInterface</hardwareInterface>
-        </joint>
-        <actuator name="joint_2_motor">
-            <hardwareInterface>hardware_interface/PositionJointInterface</hardwareInterface>
-            <mechanicalReduction>1</mechanicalReduction>
-        </actuator>
-    </transmission>
-    <transmission name="trans_joint_3">
-        <type>transmission_interface/SimpleTransmission</type>
+        <command_interface name="position">
+            <param name="min">-3.14</param>
+            <param name="max">3.14</param>
+        </command_interface>
+        <state_interface name="position">
+                <param name="initial_value">0.0</param>
+                </state_interface>
+        <state_interface name="velocity"/>
+        <state_interface name="effort"/>
+        </joint>
         <joint name="joint_3">
-            <hardwareInterface>hardware_interface/PositionJointInterface</hardwareInterface>
-        </joint>
-        <actuator name="joint_3_motor">
-            <hardwareInterface>hardware_interface/PositionJointInterface</hardwareInterface>
-            <mechanicalReduction>1</mechanicalReduction>
-        </actuator>
-    </transmission>
-    <transmission name="trans_joint_4">
-        <type>transmission_interface/SimpleTransmission</type>
+        <command_interface name="position">
+            <param name="min">-3.14</param>
+            <param name="max">3.14</param>
+        </command_interface>
+        <state_interface name="position">
+                <param name="initial_value">0.0</param>
+                </state_interface>
+        <state_interface name="velocity"/>
+        <state_interface name="effort"/>
+        </joint>
         <joint name="joint_4">
-            <hardwareInterface>hardware_interface/PositionJointInterface</hardwareInterface>
-        </joint>
-        <actuator name="joint_4_motor">
-            <hardwareInterface>hardware_interface/PositionJointInterface</hardwareInterface>
-            <mechanicalReduction>1</mechanicalReduction>
-        </actuator>
-    </transmission>
-    <transmission name="trans_joint_5">
-        <type>transmission_interface/SimpleTransmission</type>
+        <command_interface name="position">
+            <param name="min">-3.14</param>
+            <param name="max">3.14</param>
+        </command_interface>
+        <state_interface name="position">
+                <param name="initial_value">0.0</param>
+                </state_interface>
+        <state_interface name="velocity"/>
+        <state_interface name="effort"/>
+        </joint>
         <joint name="joint_5">
-            <hardwareInterface>hardware_interface/PositionJointInterface</hardwareInterface>
-        </joint>
-        <actuator name="joint_5_motor">
-            <hardwareInterface>hardware_interface/PositionJointInterface</hardwareInterface>
-            <mechanicalReduction>1</mechanicalReduction>
-        </actuator>
-    </transmission>
-    <transmission name="trans_joint_6">
-        <type>transmission_interface/SimpleTransmission</type>
+        <command_interface name="position">
+            <param name="min">-3.14</param>
+            <param name="max">3.14</param>
+        </command_interface>
+        <state_interface name="position">
+                <param name="initial_value">0.0</param>
+                </state_interface>
+        <state_interface name="velocity"/>
+        <state_interface name="effort"/>
+        </joint>
         <joint name="joint_6">
-            <hardwareInterface>hardware_interface/PositionJointInterface</hardwareInterface>
-        </joint>
-        <actuator name="joint_6_motor">
-            <hardwareInterface>hardware_interface/PositionJointInterface</hardwareInterface>
-            <mechanicalReduction>1</mechanicalReduction>
-        </actuator>
-    </transmission>
-    <gazebo reference="linear_sledge">
-        <material>Gazebo/Grey</material>
-        <mu1>0.2</mu1>
-        <mu2>0.2</mu2>
-    </gazebo>
-    <gazebo reference="link_0">
-        <material>Gazebo/Grey</material>
-        <mu1>0.2</mu1>
-        <mu2>0.2</mu2>
-    </gazebo>
-    <gazebo reference="link_1">
-        <material>Gazebo/Grey</material>
-        <mu1>0.2</mu1>
-        <mu2>0.2</mu2>
-    </gazebo>
-    <gazebo reference="link_2">
-        <material>Gazebo/Grey</material>
-        <mu1>0.2</mu1>
-        <mu2>0.2</mu2>
-    </gazebo>
-    <gazebo reference="link_3">
-        <material>Gazebo/Grey</material>
-        <mu1>0.2</mu1>
-        <mu2>0.2</mu2>
-    </gazebo>
-    <gazebo reference="link_4">
-        <material>Gazebo/Grey</material>
-        <mu1>0.2</mu1>
-        <mu2>0.2</mu2>
-    </gazebo>
-    <gazebo reference="link_5">
-        <material>Gazebo/Grey</material>
-        <mu1>0.2</mu1>
-        <mu2>0.2</mu2>
-    </gazebo>
-    <gazebo reference="link_6">
-        <material>Gazebo/Grey</material>
-        <mu1>0.2</mu1>
-        <mu2>0.2</mu2>
-    </gazebo>
-    <!--Gazebo Plugins -->
+        <command_interface name="position">
+            <param name="min">-3.14</param>
+            <param name="max">3.14</param>
+        </command_interface>
+        <state_interface name="position">
+                <param name="initial_value">0.0</param>
+                </state_interface>
+        <state_interface name="velocity"/>
+        <state_interface name="effort"/>
+        </joint>
+    </ros2_control>
     <gazebo>
-        <plugin name="control" filename="libgazebo_ros_control.so">
-        </plugin>
-    </gazebo>
-    <gazebo>
-        <plugin name = "joint_state_publisher" filename = "libgazebo_ros_joint_state_publisher.so" >
-		<jointName>linear_axis, joint_1, joint_2, joint_3, joint_4, joint_5, joint_6</jointName>
+        <plugin name="gazebo_ros2_control" filename="libgazebo_ros2_control.so">
+            <robot_sim_type>gazebo_ros2_control/GazeboSystem</robot_sim_type>
+            <parameters>$(find six_dofra_config)/config/ros2_controllers.yaml</parameters>
         </plugin>
     </gazebo>
